Commit message: changed kinect_link to kinect_mount, kinect_link is a new link

File: arips_description/urdf/arips_onshape.urdf (robot description, URDF)
Before this commit: robot arips, 13 links, 12 joints
Links:
- removed link kinect_link
- added link kinect_mount, mass 0.000665142; visual mesh filename=package://arips_description/meshes/kinect_link.gltf scale=1 1 1
Joints:
- joint fastened_2_0: parent kinect_link -> kinect_mount
- joint kinect_joint_0: child kinect_link -> kinect_mount
