Commit message: kinect servo working with new library

File: arips_description/urdf/arips.ros2_control.xacro (robot description, xacro)
@@ -1,22 +1,49 @@
 <?xml version="1.0"?>
 <robot xmlns:xacro="http://www.ros.org/wiki/xacro">
-    <xacro:macro name="ros2_control_arips" params="usb_port baudrate joint_config_file arm_enabled kinect_enabled">
+    <xacro:macro name="ros2_control_arips" params="serial_port baud_rate arm_enabled kinect_enabled">
         <ros2_control name="arips_servos" type="system">
             <hardware>
-                <plugin>feetech_ros2_driver/FeetechHardwareInterface</plugin>
-                <param name="usb_port">${usb_port}</param>
-                <!-- feetech_ros2_driver v0.2.2 ignores this and hardcodes 1,000,000 baud; kept for forward-compat -->
-                <param name="baudrate">${baudrate}</param>
-                <param name="joint_config_file">${joint_config_file}</param>
+                <plugin>sts_hardware_interface/STSHardwareInterface</plugin>
+                <param name="serial_port">${serial_port}</param>
+                <param name="baud_rate">${baud_rate}</param>
+                <param name="communication_timeout_ms">20</param>  <!-- Serial timeout: 1-1000 ms (default: 100) -->
+                <param name="use_sync_write">true</param>  <!-- Enable SyncWrite for multi-motor chains (default: true) -->
+                <param name="enable_mock_mode">false</param>  <!-- Simulation mode without hardware (default: false) -->
+                <param name="reset_states_on_activate">"false"</param>  <!-- Reset position/velocity to zero on activation (default: true) -->
             </hardware>
             <xacro:if value="${kinect_enabled}">
                 <joint name="kinect_joint_0">
-                    <param name="id">5</param>
-                    <command_interface name="position" />
-                    <state_interface name="position" />
-                    <state_interface name="velocity" />
+                    <!-- Required Joint Parameters -->
+                    <param name="motor_id">7</param>  <!-- Motor ID on serial bus: 1-253 -->
+                    <!-- Optional Joint Parameters -->
+                    <param name="operating_mode">0</param>  <!-- 0=Position, 1=Velocity, 2=PWM [default: 1] -->
+                    <param name="min_position">-1.5708</param>  <!-- Min position limit in radians (default: 0.0) -->
+                    <param name="max_position">0.0</param>
+                    <param name="max_velocity_steps">3400</param>  <!-- Motor's max velocity in steps/s, model-dependent: STS3215=3400, STS3032=2900 (default: 3400) -->
+                    <param name="max_velocity">5.22</param>  <!-- Max velocity limit in rad/s (default: 5.22) -->
+                    <param name="position_center_steps">1173</param>  <!-- Motor step mapped to 0 rad: 0-4095 (default: 4095 → [0, 2π); set to 2048 for [−π, +π]) -->
+                    <!-- Optional EEPROM parameters (omit any line to preserve the existing EEPROM value): -->
+                    <!-- <param name="p_coefficient">32</param> -->   <!-- P gain (0-255): addr 21 (Mode 0) -->
+                    <!-- <param name="d_coefficient">32</param> -->   <!-- D gain (0-255): addr 22 (Mode 0 only; ignored in Mode 1/2) -->
+                    <!-- <param name="i_coefficient">0</param> -->    <!-- I gain (0-255): addr 23 (Mode 0), addr 39 (Mode 1) -->
+                    <!-- <param name="protection_current">462</param> -->  <!-- Hardware current cutoff (0-65535, 6.5mA units; 462 ≈ 3.0A): addr 28/29 -->
+                    <!-- <param name="overload_torque">80</param> -->      <!-- Load threshold for overload protection (0-254): addr 36 -->
+                    <!-- <param name="return_delay">0</param> -->          <!-- Response delay (0-254, 2µs units): addr 7 -->
+                    <!-- <param name="deadband">2</param> -->              <!-- Position insensitive-area (0-255): addr 26/27 (CW_DEAD/CCW_DEAD), both set to the same value (Mode 0 only; ignored in Mode 1/2) -->
+                    <!-- Command Interfaces (Mode 0: Position) -->
+                    <command_interface name="position"/>  <!-- Target position in radians -->
+                    <command_interface name="velocity"/>  <!-- Max speed in rad/s -->
+                    <command_interface name="acceleration"/>  <!-- Acceleration value: 0-254 -->
+                    <!-- State Interfaces (always exported, declarations optional but recommended) -->
+                    <state_interface name="position"/>  <!-- Current position (radians) -->
+                    <state_interface name="velocity"/>  <!-- Current velocity (rad/s) -->
+                    <state_interface name="effort"/>  <!-- Motor load (-1.0 to +1.0) -->
+                    <state_interface name="voltage"/>  <!-- Supply voltage (volts) -->
+                    <state_interface name="temperature"/>  <!-- Internal temperature (°C) -->
+                    <state_interface name="current"/>  <!-- Motor current draw (amperes) -->
+                    <state_interface name="is_moving"/>  <!-- Motion status (1.0=moving, 0.0=stopped) -->
                 </joint>
             </xacro:if>
-            <xacro:if value="${arm_enabled}">
+            <!-- <xacro:if value="${arm_enabled}">
                 <joint name="revolute_2_0">
                     <param name="id">1</param>
@@ -43,5 +70,5 @@
                     <state_interface name="velocity" />
                 </joint>
-            </xacro:if>
+            </xacro:if> -->
         </ros2_control>
     </xacro:macro>

File: arips_description/urdf/arips_onshape.urdf.xacro (robot description, xacro)
@@ -2,7 +2,6 @@
 <robot name="arips" xmlns:xacro="http://www.ros.org/wiki/xacro">
     <xacro:arg name="use_ros2_control" default="false" />
-    <xacro:arg name="usb_port" default="/dev/feetech_servo" />
-    <xacro:arg name="baudrate" default="1000000" />
-    <xacro:arg name="joint_config_file" default="" />
+    <xacro:arg name="serial_port" default="/dev/feetech_servo" />
+    <xacro:arg name="baud_rate" default="1000000" />
     <xacro:arg name="arm_enabled" default="true" />
     <xacro:arg name="kinect_enabled" default="true" />
@@ -257,5 +256,5 @@
     <joint name="kinect_joint_0" type="continuous">
         <origin xyz="0.01 -0.14 1.166" rpy="2.37643e-17 1.18821e-17 6.12323e-17" />
-        <axis xyz="1 0 0" />
+        <axis xyz="-1 0 0" />
         <parent link="base_upper" />
         <child link="kinect_mount" />
@@ -287,5 +286,5 @@
     </joint>
     <xacro:if value="$(arg use_ros2_control)">
-        <xacro:ros2_control_arips usb_port="$(arg usb_port)" baudrate="$(arg baudrate)" joint_config_file="$(arg joint_config_file)" arm_enabled="$(arg arm_enabled)" kinect_enabled="$(arg kinect_enabled)" />
+        <xacro:ros2_control_arips serial_port="$(arg serial_port)" baud_rate="$(arg baud_rate)" arm_enabled="$(arg arm_enabled)" kinect_enabled="$(arg kinect_enabled)" />
     </xacro:if>
 </robot>

Commit message: new urdf file with better kinect position

File: arips_description/urdf/arips.ros2_control.xacro (robot description, xacro)
@@ -13,5 +13,5 @@
             </hardware>
             <xacro:if value="${kinect_enabled}">
-                <joint name="kinect_joint_0">
+                <joint name="kinect_joint">
                     <!-- Required Joint Parameters -->
                     <param name="motor_id">7</param>  <!-- Motor ID on serial bus: 1-253 -->

File: arips_description/urdf/arips_onshape.urdf.xacro (robot description, xacro)
@@ -16,8 +16,7 @@
             <origin xyz="0 0 0" rpy="0 -0 0" />
             <geometry>
-                <mesh filename="package://arips_description/meshes/Base lower.gltf" scale="1 1 1" />
+                <mesh filename="package://arips_description/meshes/Base_lower.gltf" scale="1 1 1" />
             </geometry>
             <material name="0.756863_0.462745_0.109804_0.000000_0.000000">
-                <texture />
                 <color rgba="0.756863 0.462745 0.109804 1" />
             </material>
@@ -26,15 +25,14 @@
     <link name="base_upper">
         <inertial>
-            <mass value="0.00167698" />
-            <origin xyz="0.033655 -0.0364095 0.313631" rpy="0 -0 0" />
-            <inertia ixx="0.000158733" ixy="5.84651e-06" ixz="-2.16466e-05" iyy="0.000158003" iyz="2.46039e-05" izz="4.27272e-05" />
-        </inertial>
-        <visual>
-            <origin xyz="0 0 0" rpy="0 -0 0" />
-            <geometry>
-                <mesh filename="package://arips_description/meshes/Base upper.gltf" scale="1 1 1" />
+            <mass value="0.00176738" />
+            <origin xyz="0.0388387 -0.0417081 0.36814" rpy="0 -0 0" />
+            <inertia ixx="0.000256556" ixy="6.74702e-06" ixz="-3.03595e-05" iyy="0.000255786" iyz="3.40732e-05" izz="4.45347e-05" />
+        </inertial>
+        <visual>
+            <origin xyz="0 0 0" rpy="0 -0 0" />
+            <geometry>
+                <mesh filename="package://arips_description/meshes/Base_upper.gltf" scale="1 1 1" />
             </geometry>
             <material name="0.756863_0.462745_0.109804_0.000000_0.000000">
-                <texture />
                 <color rgba="0.756863 0.462745 0.109804 1" />
             </material>
@@ -53,5 +51,4 @@
             </geometry>
             <material name="0.647059_0.647059_0.647059_0.000000_0.000000">
-                <texture />
                 <color rgba="0.647059 0.647059 0.647059 1" />
             </material>
@@ -61,15 +58,14 @@
         <inertial>
             <mass value="0.000375246" />
-            <origin xyz="-2.02802e-19 -0.651131 -4.44089e-16" rpy="0 -0 0" />
+            <origin xyz="-1.93985e-19 -0.651131 -6.66134e-16" rpy="0 -0 0" />
             <inertia ixx="2.85294e-05" ixy="0" ixz="0" iyy="8.56168e-06" iyz="0" izz="1.99677e-05" />
         </inertial>
         <visual>
-            <origin xyz="0 0.1725 -1.216" rpy="0 -0 0" />
-            <geometry>
-                <mesh filename="package://arips_description/meshes/Kinect beam.gltf" scale="1 1 1" />
-            </geometry>
-            <material name="0.341176_0.776471_0.741176_0.000000_0.901961">
-                <texture />
-                <color rgba="0.341176 0.776471 0.741176 0.0980392" />
+            <origin xyz="0 0.1725 -1.442" rpy="0 -0 0" />
+            <geometry>
+                <mesh filename="package://arips_description/meshes/Kinect_beam.gltf" scale="1 1 1" />
+            </geometry>
+            <material name="0.341176_0.776471_0.741176_0.000000_0.000000">
+                <color rgba="0.341176 0.776471 0.741176 0.1" />
             </material>
         </visual>
@@ -82,10 +78,9 @@
         </inertial>
         <visual>
-            <origin xyz="-0.01 0.14 -1.166" rpy="0 -0 0" />
-            <geometry>
-                <mesh filename="package://arips_description/meshes/kinect_link.gltf" scale="1 1 1" />
+            <origin xyz="-0.01 0.14 -1.392" rpy="0 -0 0" />
+            <geometry>
+                <mesh filename="package://arips_description/meshes/kinect_mount.gltf" scale="1 1 1" />
             </geometry>
             <material name="0.156863_0.156863_0.156863_0.000000_0.000000">
-                <texture />
                 <color rgba="0.156863 0.156863 0.156863 1" />
             </material>
@@ -95,14 +90,13 @@
         <inertial>
             <mass value="0.00232688" />
-            <origin xyz="-4.65948e-17 7.63278e-17 -0.0125" rpy="0 -0 0" />
+            <origin xyz="0 2.94903e-17 -0.0125" rpy="0 -0 0" />
             <inertia ixx="1.27299e-05" ixy="0" ixz="0" iyy="2.59544e-05" iyz="0" izz="3.84419e-05" />
         </inertial>
         <visual>
-            <origin xyz="-3.72758e-17 -0.00848802 -0.201" rpy="0 -0 0" />
+            <origin xyz="0 -0.00848802 -0.201" rpy="0 -0 0" />
             <geometry>
                 <mesh filename="package://arips_description/meshes/Laptop.gltf" scale="1 1 1" />
             </geometry>
             <material name="0.156863_0.156863_0.156863_0.000000_0.000000">
-                <texture />
                 <color rgba="0.156863 0.156863 0.156863 1" />
             </material>
@@ -118,8 +112,7 @@
             <origin xyz="-0.125 0.13 -0.676" rpy="0 -0 0" />
             <geometry>
-                <mesh filename="package://arips_description/meshes/Link 0.gltf" scale="1 1 1" />
+                <mesh filename="package://arips_description/meshes/Link_0.gltf" scale="1 1 1" />
             </geometry>
             <material name="0.498039_0.498039_0.498039_0.000000_0.000000">
-                <texture />
                 <color rgba="0.498039 0.498039 0.498039 1" />
             </material>
@@ -135,8 +128,7 @@
             <origin xyz="-0.1 0.14 -0.676" rpy="0 -0 0" />
             <geometry>
-                <mesh filename="package://arips_description/meshes/Link 1.gltf" scale="1 1 1" />
+                <mesh filename="package://arips_description/meshes/Link_1.gltf" scale="1 1 1" />
             </geometry>
             <material name="0.980392_0.713725_0.003922_0.000000_0.000000">
-                <texture />
                 <color rgba="0.980392 0.713726 0.00392157 1" />
             </material>
@@ -152,8 +144,7 @@
             <origin xyz="0.07 0.14 -0.666" rpy="0 -0 0" />
             <geometry>
-                <mesh filename="package://arips_description/meshes/Link 2.gltf" scale="1 1 1" />
+                <mesh filename="package://arips_description/meshes/Link_2.gltf" scale="1 1 1" />
             </geometry>
             <material name="0.615686_0.811765_0.929412_0.000000_0.000000">
-                <texture />
                 <color rgba="0.615686 0.811765 0.929412 1" />
             </material>
@@ -169,8 +160,7 @@
             <origin xyz="0.07 -0.01 -0.656" rpy="0 -0 0" />
             <geometry>
-                <mesh filename="package://arips_description/meshes/Link 3.gltf" scale="1 1 1" />
+                <mesh filename="package://arips_description/meshes/Link_3.gltf" scale="1 1 1" />
             </geometry>
             <material name="0.647059_0.647059_0.647059_0.000000_0.000000">
-                <texture />
                 <color rgba="0.647059 0.647059 0.647059 1" />
             </material>
@@ -187,8 +177,7 @@
             <origin xyz="0 0 0" rpy="0 -0 0" />
             <geometry>
-                <mesh filename="package://arips_description/meshes/Wheel left.gltf" scale="1 1 1" />
+                <mesh filename="package://arips_description/meshes/Wheel_left.gltf" scale="1 1 1" />
             </geometry>
             <material name="0.141176_0.694118_0.650980_0.000000_0.000000">
-                <texture />
                 <color rgba="0.141176 0.694118 0.65098 1" />
             </material>
@@ -204,13 +193,12 @@
             <origin xyz="0 0 0" rpy="0 -0 0" />
             <geometry>
-                <mesh filename="package://arips_description/meshes/Wheel right.gltf" scale="1 1 1" />
+                <mesh filename="package://arips_description/meshes/Wheel_right.gltf" scale="1 1 1" />
             </geometry>
             <material name="0.141176_0.694118_0.650980_0.000000_0.000000">
-                <texture />
                 <color rgba="0.141176 0.694118 0.65098 1" />
             </material>
         </visual>
     </link>
-    <joint name="fastened_1_0" type="fixed">
+    <joint name="fastened_1" type="fixed">
         <origin xyz="-1.38778e-17 0 -0.2" rpy="-5.2711e-82 -3.08149e-33 3.42114e-49" />
         <axis xyz="0 0 1" />
@@ -218,5 +206,5 @@
         <child link="gripper" />
     </joint>
-    <joint name="fastened_2_0" type="fixed">
+    <joint name="fastened_2" type="fixed">
         <origin xyz="-0.01 -0.0325 0.05" rpy="5.55112e-17 -1.38667e-32 -3.04851e-32" />
         <axis xyz="0 -1 0" />
@@ -224,11 +212,11 @@
         <child link="kinect_beam" />
     </joint>
-    <joint name="fastened_4_0" type="fixed">
+    <joint name="fastened_4" type="fixed">
         <origin xyz="-0.000349049 0.000361977 0.176" rpy="3.14159 -0 0" />
-        <axis xyz="0 0 -1" />
+        <axis xyz="-0 -0 1" />
         <parent link="base_upper" />
         <child link="laptop" />
     </joint>
-    <joint name="fastened_5_0" type="fixed">
+    <joint name="fastened_5" type="fixed">
         <origin xyz="0 0 0" rpy="0 -0 0" />
         <axis xyz="0 0 1" />
@@ -236,5 +224,5 @@
         <child link="wheel_left" />
     </joint>
-    <joint name="fastened_6_0" type="fixed">
+    <joint name="fastened_6" type="fixed">
         <origin xyz="0 0 0" rpy="0 -0 0" />
         <axis xyz="0 0 1" />
@@ -242,5 +230,5 @@
         <child link="wheel_right" />
     </joint>
-    <joint name="fastened_7_0" type="fixed">
+    <joint name="fastened_7" type="fixed">
         <origin xyz="0 0 0" rpy="0 -0 0" />
         <axis xyz="0 0 1" />
@@ -248,5 +236,5 @@
         <child link="base_upper" />
     </joint>
-    <joint name="fastened_8_0" type="fixed">
+    <joint name="fastened_8" type="fixed">
         <origin xyz="0 0 0" rpy="0 -0 1.5708" />
         <axis xyz="0 0 1" />
@@ -254,34 +242,36 @@
         <child link="base_lower" />
     </joint>
-    <joint name="kinect_joint_0" type="continuous">
-        <origin xyz="0.01 -0.14 1.166" rpy="2.37643e-17 1.18821e-17 6.12323e-17" />
+    <joint name="kinect_joint" type="continuous">
+        <origin xyz="0.01 -0.14 1.392" rpy="2.37643e-17 1.18821e-17 6.12323e-17" />
         <axis xyz="-1 0 0" />
         <parent link="base_upper" />
         <child link="kinect_mount" />
     </joint>
-    <joint name="revolute_2_0" type="continuous">
+    <joint name="revolute_2" type="revolute">
         <origin xyz="-0.0191667 -0.01 0" rpy="-5.5358e-20 -5.84736e-19 0.290951" />
-        <axis xyz="0 0 -1" />
+        <axis xyz="-0 -0 1" />
         <parent link="link_0" />
         <child link="link_1" />
-    </joint>
-    <joint name="revolute_3_0" type="continuous">
+        <limit effort="1" velocity="1" lower="-2.64715" upper="2.06524" />
+    </joint>
+    <joint name="revolute_3" type="revolute">
         <origin xyz="-0.17 1.11022e-16 -0.01" rpy="1.55162e-24 -8.5589e-24 -2.38997" />
-        <axis xyz="0 0 -1" />
+        <axis xyz="-0 -0 1" />
         <parent link="link_1" />
         <child link="link_2" />
-    </joint>
-    <joint name="revolute_4_0" type="continuous">
+        <limit effort="1" velocity="1" lower="-4.67861" upper="0.033776" />
+    </joint>
+    <joint name="revolute_4" type="continuous">
         <origin xyz="-2.77556e-17 0.15 -0.01" rpy="-4.29773e-17 4.29663e-17 -1.0386" />
-        <axis xyz="0 0 -1" />
+        <axis xyz="-0 -0 1" />
         <parent link="link_2" />
         <child link="link_3" />
     </joint>
-    <joint name="slider_1_0" type="prismatic">
+    <joint name="slider_1" type="prismatic">
         <origin xyz="0.125 -0.13 0.518053" rpy="4.32978e-17 -6.16298e-33 3.88263e-34" />
         <axis xyz="0 0 1" />
         <parent link="base_upper" />
         <child link="link_0" />
-        <limit effort="1" velocity="1" lower="-0.5" upper="0.5" />
+        <limit effort="1" velocity="1" lower="-0.332053" upper="0.657947" />
     </joint>
     <xacro:if value="$(arg use_ros2_control)">
