Commit message: WIP make most arm joints work

File: arips_description/urdf/arips.ros2_control.xacro (robot description, xacro)
@@ -8,5 +8,5 @@
                 <param name="baud_rate">${baud_rate}</param>
                 <param name="communication_timeout_ms">20</param>  <!-- Serial timeout: 1-1000 ms (default: 100) -->
-                <param name="use_sync_write">true</param>  <!-- Enable SyncWrite for multi-motor chains (default: true) -->
+                <param name="use_sync_write">false</param>  <!-- Enable SyncWrite for multi-motor chains (default: true) -->
                 <param name="enable_mock_mode">false</param>  <!-- Simulation mode without hardware (default: false) -->
                 <param name="reset_states_on_activate">"false"</param>  <!-- Reset position/velocity to zero on activation (default: true) -->
@@ -45,30 +45,122 @@
                 </joint>
             </xacro:if>
-            <!-- <xacro:if value="${arm_enabled}">
-                <joint name="revolute_2_0">
-                    <param name="id">1</param>
-                    <command_interface name="position" />
-                    <state_interface name="position" />
-                    <state_interface name="velocity" />
+             <xacro:if value="${arm_enabled}">
+                <joint name="revolute_2">
+                    <!-- Required Joint Parameters -->
+                    <param name="motor_id">2</param>  <!-- Motor ID on serial bus: 1-253 -->
+                    <!-- Optional Joint Parameters -->
+                    <param name="operating_mode">0</param>  <!-- 0=Position, 1=Velocity, 2=PWM [default: 1] -->
+                    <param name="min_position">-3.1416</param>  <!-- Min position limit in radians (default: 0.0) -->
+                    <param name="max_position">3.1416</param>  <!-- Max position limit in radians (default: 0.0) -->
+                    <param name="max_velocity_steps">3400</param>  <!-- Motor's max velocity in steps/s, model-dependent: STS3215=3400, STS3032=2900 (default: 3400) -->
+                    <param name="max_velocity">5.22</param>  <!-- Max velocity limit in rad/s (default: 5.22) -->
+                    <param name="position_center_steps">2048</param>  <!-- Motor step mapped to 0 rad: 0-4095 (default: 4095 → [0, 2π); set to 2048 for [−π, +π]) -->
+                    <!-- Optional EEPROM parameters (omit any line to preserve the existing EEPROM value): -->
+                    <!-- <param name="p_coefficient">32</param> -->   <!-- P gain (0-255): addr 21 (Mode 0) -->
+                    <!-- <param name="d_coefficient">32</param> -->   <!-- D gain (0-255): addr 22 (Mode 0 only; ignored in Mode 1/2) -->
+                    <!-- <param name="i_coefficient">0</param> -->    <!-- I gain (0-255): addr 23 (Mode 0), addr 39 (Mode 1) -->
+                    <!-- <param name="protection_current">462</param> -->  <!-- Hardware current cutoff (0-65535, 6.5mA units; 462 ≈ 3.0A): addr 28/29 -->
+                    <!-- <param name="overload_torque">80</param> -->      <!-- Load threshold for overload protection (0-254): addr 36 -->
+                    <!-- <param name="return_delay">0</param> -->          <!-- Response delay (0-254, 2µs units): addr 7 -->
+                    <!-- <param name="deadband">2</param> -->              <!-- Position insensitive-area (0-255): addr 26/27 (CW_DEAD/CCW_DEAD), both set to the same value (Mode 0 only; ignored in Mode 1/2) -->
+                    <!-- Command Interfaces (Mode 0: Position) -->
+                    <command_interface name="position"/>  <!-- Target position in radians -->
+                    <command_interface name="velocity"/>  <!-- Max speed in rad/s -->
+                    <command_interface name="acceleration"/>  <!-- Acceleration value: 0-254 -->
+                    <!-- State Interfaces (always exported, declarations optional but recommended) -->
+                    <state_interface name="position"/>  <!-- Current position (radians) -->
+                    <state_interface name="velocity"/>  <!-- Current velocity (rad/s) -->
+                    <state_interface name="effort"/>  <!-- Motor load (-1.0 to +1.0) -->
+                    <state_interface name="voltage"/>  <!-- Supply voltage (volts) -->
+                    <state_interface name="temperature"/>  <!-- Internal temperature (°C) -->
+                    <state_interface name="current"/>  <!-- Motor current draw (amperes) -->
+                    <state_interface name="is_moving"/>  <!-- Motion status (1.0=moving, 0.0=stopped) -->
                 </joint>
-                <joint name="revolute_3_0">
-                    <param name="id">2</param>
-                    <command_interface name="position" />
-                    <state_interface name="position" />
-                    <state_interface name="velocity" />
+                <joint name="revolute_3">
+                   <!-- Required Joint Parameters -->
+                    <param name="motor_id">3</param>  <!-- Motor ID on serial bus: 1-253 -->
+                    <!-- Optional Joint Parameters -->
+                    <param name="operating_mode">0</param>  <!-- 0=Position, 1=Velocity, 2=PWM [default: 1] -->
+                    <param name="min_position">-3.1416</param>  <!-- Min position limit in radians (default: 0.0) -->
+                    <param name="max_position">3.1416</param>  <!-- Max position limit in radians (default: 0.0) -->
+                    <param name="max_velocity_steps">3400</param>  <!-- Motor's max velocity in steps/s, model-dependent: STS3215=3400, STS3032=2900 (default: 3400) -->
+                    <param name="max_velocity">5.22</param>  <!-- Max velocity limit in rad/s (default: 5.22) -->
+                    <param name="position_center_steps">2048</param>  <!-- Motor step mapped to 0 rad: 0-4095 (default: 4095 → [0, 2π); set to 2048 for [−π, +π]) -->
+                    <!-- Optional EEPROM parameters (omit any line to preserve the existing EEPROM value): -->
+                    <!-- <param name="p_coefficient">32</param> -->   <!-- P gain (0-255): addr 21 (Mode 0) -->
+                    <!-- <param name="d_coefficient">32</param> -->   <!-- D gain (0-255): addr 22 (Mode 0 only; ignored in Mode 1/2) -->
+                    <!-- <param name="i_coefficient">0</param> -->    <!-- I gain (0-255): addr 23 (Mode 0), addr 39 (Mode 1) -->
+                    <!-- <param name="protection_current">462</param> -->  <!-- Hardware current cutoff (0-65535, 6.5mA units; 462 ≈ 3.0A): addr 28/29 -->
+                    <!-- <param name="overload_torque">80</param> -->      <!-- Load threshold for overload protection (0-254): addr 36 -->
+                    <!-- <param name="return_delay">0</param> -->          <!-- Response delay (0-254, 2µs units): addr 7 -->
+                    <!-- <param name="deadband">2</param> -->              <!-- Position insensitive-area (0-255): addr 26/27 (CW_DEAD/CCW_DEAD), both set to the same value (Mode 0 only; ignored in Mode 1/2) -->
+                    <!-- Command Interfaces (Mode 0: Position) -->
+                    <command_interface name="position"/>  <!-- Target position in radians -->
+                    <command_interface name="velocity"/>  <!-- Max speed in rad/s -->
+                    <command_interface name="acceleration"/>  <!-- Acceleration value: 0-254 -->
+                    <!-- State Interfaces (always exported, declarations optional but recommended) -->
+                    <state_interface name="position"/>  <!-- Current position (radians) -->
+                    <state_interface name="velocity"/>  <!-- Current velocity (rad/s) -->
+                    <state_interface name="effort"/>  <!-- Motor load (-1.0 to +1.0) -->
+                    <state_interface name="voltage"/>  <!-- Supply voltage (volts) -->
+                    <state_interface name="temperature"/>  <!-- Internal temperature (°C) -->
+                    <state_interface name="current"/>  <!-- Motor current draw (amperes) -->
+                    <state_interface name="is_moving"/>  <!-- Motion status (1.0=moving, 0.0=stopped) -->
                 </joint>
-                <joint name="revolute_4_0">
-                    <param name="id">3</param>
-                    <command_interface name="position" />
-                    <state_interface name="position" />
-                    <state_interface name="velocity" />
+                <joint name="revolute_4">
+                   <!-- Required Joint Parameters -->
+                    <param name="motor_id">4</param>  <!-- Motor ID on serial bus: 1-253 -->
+                    <!-- Optional Joint Parameters -->
+                    <param name="operating_mode">0</param>  <!-- 0=Position, 1=Velocity, 2=PWM [default: 1] -->
+                    <param name="min_position">-3.1416</param>  <!-- Min position limit in radians (default: 0.0) -->
+                    <param name="max_position">3.1416</param>  <!-- Max position limit in radians (default: 0.0) -->
+                    <param name="max_velocity_steps">3400</param>  <!-- Motor's max velocity in steps/s, model-dependent: STS3215=3400, STS3032=2900 (default: 3400) -->
+                    <param name="max_velocity">5.22</param>  <!-- Max velocity limit in rad/s (default: 5.22) -->
+                    <param name="position_center_steps">2048</param>  <!-- Motor step mapped to 0 rad: 0-4095 (default: 4095 → [0, 2π); set to 2048 for [−π, +π]) -->
+                    <!-- Optional EEPROM parameters (omit any line to preserve the existing EEPROM value): -->
+                    <!-- <param name="p_coefficient">32</param> -->   <!-- P gain (0-255): addr 21 (Mode 0) -->
+                    <!-- <param name="d_coefficient">32</param> -->   <!-- D gain (0-255): addr 22 (Mode 0 only; ignored in Mode 1/2) -->
+                    <!-- <param name="i_coefficient">0</param> -->    <!-- I gain (0-255): addr 23 (Mode 0), addr 39 (Mode 1) -->
+                    <!-- <param name="protection_current">462</param> -->  <!-- Hardware current cutoff (0-65535, 6.5mA units; 462 ≈ 3.0A): addr 28/29 -->
+                    <!-- <param name="overload_torque">80</param> -->      <!-- Load threshold for overload protection (0-254): addr 36 -->
+                    <!-- <param name="return_delay">0</param> -->          <!-- Response delay (0-254, 2µs units): addr 7 -->
+                    <!-- <param name="deadband">2</param> -->              <!-- Position insensitive-area (0-255): addr 26/27 (CW_DEAD/CCW_DEAD), both set to the same value (Mode 0 only; ignored in Mode 1/2) -->
+                    <!-- Command Interfaces (Mode 0: Position) -->
+                    <command_interface name="position"/>  <!-- Target position in radians -->
+                    <command_interface name="velocity"/>  <!-- Max speed in rad/s -->
+                    <command_interface name="acceleration"/>  <!-- Acceleration value: 0-254 -->
+                    <!-- State Interfaces (always exported, declarations optional but recommended) -->
+                    <state_interface name="position"/>  <!-- Current position (radians) -->
+                    <state_interface name="velocity"/>  <!-- Current velocity (rad/s) -->
+                    <state_interface name="effort"/>  <!-- Motor load (-1.0 to +1.0) -->
+                    <state_interface name="voltage"/>  <!-- Supply voltage (volts) -->
+                    <state_interface name="temperature"/>  <!-- Internal temperature (°C) -->
+                    <state_interface name="current"/>  <!-- Motor current draw (amperes) -->
+                    <state_interface name="is_moving"/>  <!-- Motion status (1.0=moving, 0.0=stopped) -->
                 </joint>
-                <joint name="slider_1_0">
-                    <param name="id">6</param>
-                    <command_interface name="position" />
-                    <state_interface name="position" />
-                    <state_interface name="velocity" />
+                <joint name="slider_1">
+                    <!-- Required Joint Parameters -->
+                    <param name="motor_id">1</param>  <!-- Motor ID on serial bus: 1-253 -->
+                    <!-- Optional Joint Parameters -->
+                    <param name="operating_mode">0</param>  <!-- 0=Position, 1=Velocity, 2=PWM [default: 1] -->
+                    <param name="min_position">0</param>  <!-- Min position limit in radians (default: 0.0) -->
+                    <param name="max_position">6.28</param>
+                    <param name="max_velocity_steps">3400</param>  <!-- Motor's max velocity in steps/s, model-dependent: STS3215=3400, STS3032=2900 (default: 3400) -->
+                    <param name="max_velocity">5.22</param>  <!-- Max velocity limit in rad/s (default: 5.22) -->
+                    <param name="position_center_steps">4095</param>  <!-- Motor step mapped to 0 rad: 0-4095 (default: 4095 → [0, 2π); set to 2048 for [−π, +π]) -->
+                    <!-- Optional EEPROM parameters (omit any line to preserve the existing EEPROM value): -->
+                    <!-- <param name="p_coefficient">32</param> -->   <!-- P gain (0-255): addr 21 (Mode 0) -->
+                    <!-- <param name="d_coefficient">32</param> -->   <!-- D gain (0-255): addr 22 (Mode 0 only; ignored in Mode 1/2) -->
+                    <!-- <param name="i_coefficient">0</param> -->    <!-- I gain (0-255): addr 23 (Mode 0), addr 39 (Mode 1) -->
+                    <!-- <param name="protection_current">462</param> -->  <!-- Hardware current cutoff (0-65535, 6.5mA units; 462 ≈ 3.0A): addr 28/29 -->
+                    <!-- <param name="overload_torque">80</param> -->      <!-- Load threshold for overload protection (0-254): addr 36 -->
+                    <!-- <param name="return_delay">0</param> -->          <!-- Response delay (0-254, 2µs units): addr 7 -->
+                    <!-- <param name="deadband">2</param> -->              <!-- Position insensitive-area (0-255): addr 26/27 (CW_DEAD/CCW_DEAD), both set to the same value (Mode 0 only; ignored in Mode 1/2) -->
+                    <!-- Command Interfaces (Mode 0: Position) -->
+                    <command_interface name="position"/>  <!-- Target position in radians -->
+                    <!-- State Interfaces (always exported, declarations optional but recommended) -->
+                    <state_interface name="position"/>  <!-- Current position (radians) -->
                 </joint>
-            </xacro:if> -->
+            </xacro:if>
         </ros2_control>
     </xacro:macro>

File: arips_description/urdf/arips_onshape.urdf.xacro (robot description, xacro)
@@ -3,5 +3,5 @@
     <xacro:arg name="use_ros2_control" default="false" />
     <xacro:arg name="serial_port" default="/dev/feetech_servo" />
-    <xacro:arg name="baud_rate" default="1000000" />
+    <xacro:arg name="baud_rate" default="500000" />
     <xacro:arg name="arm_enabled" default="true" />
     <xacro:arg name="kinect_enabled" default="true" />
@@ -249,22 +249,23 @@
     </joint>
     <joint name="revolute_2" type="revolute">
-        <origin xyz="-0.0191667 -0.01 0" rpy="-5.5358e-20 -5.84736e-19 0.290951" />
+        <origin xyz="-0.0191667 -0.01 0" rpy="0.0 0.0 0.0" />
         <axis xyz="-0 -0 1" />
         <parent link="link_0" />
         <child link="link_1" />
-        <limit effort="1" velocity="1" lower="-2.64715" upper="2.06524" />
+        <limit effort="1" velocity="1" lower="-2.3" upper="2.3" />
     </joint>
     <joint name="revolute_3" type="revolute">
-        <origin xyz="-0.17 1.11022e-16 -0.01" rpy="1.55162e-24 -8.5589e-24 -2.38997" />
+        <origin xyz="-0.17 1.11022e-16 -0.01" rpy="0.0 0.0 1.5708" />
         <axis xyz="-0 -0 1" />
         <parent link="link_1" />
         <child link="link_2" />
-        <limit effort="1" velocity="1" lower="-4.67861" upper="0.033776" />
+        <limit effort="1" velocity="1" lower="-2.3" upper="2.3" />
     </joint>
     <joint name="revolute_4" type="continuous">
-        <origin xyz="-2.77556e-17 0.15 -0.01" rpy="-4.29773e-17 4.29663e-17 -1.0386" />
+        <origin xyz="-2.77556e-17 0.15 -0.01" rpy="0.0 0.0 0.0" />
         <axis xyz="-0 -0 1" />
         <parent link="link_2" />
         <child link="link_3" />
+        <limit effort="1" velocity="1" lower="-2.3" upper="2.3" />
     </joint>
     <joint name="slider_1" type="prismatic">
@@ -273,5 +274,5 @@
         <parent link="base_upper" />
         <child link="link_0" />
-        <limit effort="1" velocity="1" lower="-0.332053" upper="0.657947" />
+        <limit effort="1" velocity="1" lower="0.0" upper="6.0" />
     </joint>
     <xacro:if value="$(arg use_ros2_control)">
