Commit message: new with correct joint dimensions and collisions

File: arips_description/urdf/arips.ros2_control.xacro (robot description, xacro)
@@ -18,6 +18,6 @@
                     <!-- Optional Joint Parameters -->
                     <param name="operating_mode">0</param>  <!-- 0=Position, 1=Velocity, 2=PWM [default: 1] -->
-                    <param name="min_position">-1.5708</param>  <!-- Min position limit in radians (default: 0.0) -->
-                    <param name="max_position">0.0</param>
+                    <param name="min_position">-1.65806</param>  <!-- Min position limit in radians (default: 0.0) -->
+                    <param name="max_position">0.5236</param>
                     <param name="max_velocity_steps">3400</param>  <!-- Motor's max velocity in steps/s, model-dependent: STS3215=3400, STS3032=2900 (default: 3400) -->
                     <param name="max_velocity">5.22</param>  <!-- Max velocity limit in rad/s (default: 5.22) -->
@@ -46,11 +46,11 @@
             </xacro:if>
              <xacro:if value="${arm_enabled}">
-                <joint name="revolute_2">
+                <joint name="joint_2">
                     <!-- Required Joint Parameters -->
                     <param name="motor_id">2</param>  <!-- Motor ID on serial bus: 1-253 -->
                     <!-- Optional Joint Parameters -->
                     <param name="operating_mode">0</param>  <!-- 0=Position, 1=Velocity, 2=PWM [default: 1] -->
-                    <param name="min_position">-3.1416</param>  <!-- Min position limit in radians (default: 0.0) -->
-                    <param name="max_position">3.1416</param>  <!-- Max position limit in radians (default: 0.0) -->
+                    <param name="min_position">-2.26893</param>  <!-- Min position limit in radians (default: 0.0) -->
+                    <param name="max_position">2.26893</param>  <!-- Max position limit in radians (default: 0.0) -->
                     <param name="max_velocity_steps">3400</param>  <!-- Motor's max velocity in steps/s, model-dependent: STS3215=3400, STS3032=2900 (default: 3400) -->
                     <param name="max_velocity">5.22</param>  <!-- Max velocity limit in rad/s (default: 5.22) -->
@@ -77,11 +77,11 @@
                     <state_interface name="is_moving"/>  <!-- Motion status (1.0=moving, 0.0=stopped) -->
                 </joint>
-                <joint name="revolute_3">
+                <joint name="joint_3">
                    <!-- Required Joint Parameters -->
                     <param name="motor_id">3</param>  <!-- Motor ID on serial bus: 1-253 -->
                     <!-- Optional Joint Parameters -->
                     <param name="operating_mode">0</param>  <!-- 0=Position, 1=Velocity, 2=PWM [default: 1] -->
-                    <param name="min_position">-3.1416</param>  <!-- Min position limit in radians (default: 0.0) -->
-                    <param name="max_position">3.1416</param>  <!-- Max position limit in radians (default: 0.0) -->
+                    <param name="min_position">-2.44346</param>  <!-- Min position limit in radians (default: 0.0) -->
+                    <param name="max_position">2.44346</param>  <!-- Max position limit in radians (default: 0.0) -->
                     <param name="max_velocity_steps">3400</param>  <!-- Motor's max velocity in steps/s, model-dependent: STS3215=3400, STS3032=2900 (default: 3400) -->
                     <param name="max_velocity">5.22</param>  <!-- Max velocity limit in rad/s (default: 5.22) -->
@@ -108,11 +108,11 @@
                     <state_interface name="is_moving"/>  <!-- Motion status (1.0=moving, 0.0=stopped) -->
                 </joint>
-                <joint name="revolute_4">
+                <joint name="joint_4">
                    <!-- Required Joint Parameters -->
                     <param name="motor_id">4</param>  <!-- Motor ID on serial bus: 1-253 -->
                     <!-- Optional Joint Parameters -->
                     <param name="operating_mode">0</param>  <!-- 0=Position, 1=Velocity, 2=PWM [default: 1] -->
-                    <param name="min_position">-3.1416</param>  <!-- Min position limit in radians (default: 0.0) -->
-                    <param name="max_position">3.1416</param>  <!-- Max position limit in radians (default: 0.0) -->
+                    <param name="min_position">-2.0944</param>  <!-- Min position limit in radians (default: 0.0) -->
+                    <param name="max_position">2.0944</param>  <!-- Max position limit in radians (default: 0.0) -->
                     <param name="max_velocity_steps">3400</param>  <!-- Motor's max velocity in steps/s, model-dependent: STS3215=3400, STS3032=2900 (default: 3400) -->
                     <param name="max_velocity">5.22</param>  <!-- Max velocity limit in rad/s (default: 5.22) -->
@@ -139,14 +139,37 @@
                     <state_interface name="is_moving"/>  <!-- Motion status (1.0=moving, 0.0=stopped) -->
                 </joint>
-                <joint name="slider_1">
+                <joint name="joint_slider">
                     <!-- Required Joint Parameters -->
                     <param name="motor_id">1</param>  <!-- Motor ID on serial bus: 1-253 -->
                     <!-- Optional Joint Parameters -->
                     <param name="operating_mode">0</param>  <!-- 0=Position, 1=Velocity, 2=PWM [default: 1] -->
-                    <param name="min_position">0</param>  <!-- Min position limit in radians (default: 0.0) -->
-                    <param name="max_position">6.28</param>
+                    <param name="min_position">0.0</param>  <!-- Min position limit in radians (default: 0.0) -->
+                    <param name="max_position">0.871</param>
                     <param name="max_velocity_steps">3400</param>  <!-- Motor's max velocity in steps/s, model-dependent: STS3215=3400, STS3032=2900 (default: 3400) -->
                     <param name="max_velocity">5.22</param>  <!-- Max velocity limit in rad/s (default: 5.22) -->
                     <param name="position_center_steps">4095</param>  <!-- Motor step mapped to 0 rad: 0-4095 (default: 4095 → [0, 2π); set to 2048 for [−π, +π]) -->
+                    <!-- Optional EEPROM parameters (omit any line to preserve the existing EEPROM value): -->
+                    <!-- <param name="p_coefficient">32</param> -->   <!-- P gain (0-255): addr 21 (Mode 0) -->
+                    <!-- <param name="d_coefficient">32</param> -->   <!-- D gain (0-255): addr 22 (Mode 0 only; ignored in Mode 1/2) -->
+                    <!-- <param name="i_coefficient">0</param> -->    <!-- I gain (0-255): addr 23 (Mode 0), addr 39 (Mode 1) -->
+                    <!-- <param name="protection_current">462</param> -->  <!-- Hardware current cutoff (0-65535, 6.5mA units; 462 ≈ 3.0A): addr 28/29 -->
+                    <!-- <param name="overload_torque">80</param> -->      <!-- Load threshold for overload protection (0-254): addr 36 -->
+                    <!-- <param name="return_delay">0</param> -->          <!-- Response delay (0-254, 2µs units): addr 7 -->
+                    <!-- <param name="deadband">2</param> -->              <!-- Position insensitive-area (0-255): addr 26/27 (CW_DEAD/CCW_DEAD), both set to the same value (Mode 0 only; ignored in Mode 1/2) -->
+                    <!-- Command Interfaces (Mode 0: Position) -->
+                    <command_interface name="position"/>  <!-- Target position in radians -->
+                    <!-- State Interfaces (always exported, declarations optional but recommended) -->
+                    <state_interface name="position"/>  <!-- Current position (radians) -->
+                </joint>
+                <joint name="joint_door_gripper">
+                    <!-- Required Joint Parameters -->
+                    <param name="motor_id">5</param>  <!-- Motor ID on serial bus: 1-253 -->
+                    <!-- Optional Joint Parameters -->
+                    <param name="operating_mode">0</param>  <!-- 0=Position, 1=Velocity, 2=PWM [default: 1] -->
+                    <param name="min_position">-3.1416</param>  <!-- Min position limit in radians (default: 0.0) -->
+                    <param name="max_position">3.1416</param>
+                    <param name="max_velocity_steps">3400</param>  <!-- Motor's max velocity in steps/s, model-dependent: STS3215=3400, STS3032=2900 (default: 3400) -->
+                    <param name="max_velocity">5.22</param>  <!-- Max velocity limit in rad/s (default: 5.22) -->
+                    <param name="position_center_steps">2048</param>  <!-- Motor step mapped to 0 rad: 0-4095 (default: 4095 → [0, 2π); set to 2048 for [−π, +π]) -->
                     <!-- Optional EEPROM parameters (omit any line to preserve the existing EEPROM value): -->
                     <!-- <param name="p_coefficient">32</param> -->   <!-- P gain (0-255): addr 21 (Mode 0) -->
