Commit message: new with correct joint dimensions and collisions

File: arips_description/urdf/arips_onshape.urdf.xacro (robot description, xacro)
@@ -1,4 +1,4 @@
-<!--URDF generated by ONSHAPE BY PTC INC, 1.213-->
-<robot name="arips" xmlns:xacro="http://www.ros.org/wiki/xacro">
+<!--URDF generated by ONSHAPE BY PTC INC, 1.222-->
+<robot name="arips_description" xmlns:xacro="http://www.ros.org/wiki/xacro">
     <xacro:arg name="use_ros2_control" default="false" />
     <xacro:arg name="serial_port" default="/dev/feetech_servo" />
@@ -7,14 +7,30 @@
     <xacro:arg name="kinect_enabled" default="true" />
     <xacro:include filename="$(find arips_description)/urdf/arips.ros2_control.xacro" />
-    <link name="base_lower">
-        <inertial>
-            <mass value="0.00124085" />
-            <origin xyz="2.01511e-18 2.73049e-18 0.114" rpy="0 -0 0" />
-            <inertia ixx="1.53964e-05" ixy="0" ixz="0" iyy="1.53964e-05" iyz="0" izz="3.07796e-05" />
-        </inertial>
-        <visual>
-            <origin xyz="0 0 0" rpy="0 -0 0" />
-            <geometry>
-                <mesh filename="package://arips_description/meshes/Base_lower.stl" scale="1 1 1" />
+    <link name="alu">
+        <inertial>
+            <mass value="0.0005768" />
+            <origin xyz="0.14 0.111595 0.904595" rpy="0 -0 0" />
+            <inertia ixx="8.68884e-05" ixy="0" ixz="0" iyy="8.48644e-05" iyz="6.53947e-06" izz="2.06249e-06" />
+        </inertial>
+        <visual>
+            <origin xyz="0 0 0" rpy="0 -0 0" />
+            <geometry>
+                <mesh filename="package://arips_description/meshes/Alu.stl" scale="1 1 1" />
+            </geometry>
+            <material name="0.156863_0.156863_0.156863_0.000000_0.000000">
+                <color rgba="0.156863 0.156863 0.156863 1" />
+            </material>
+        </visual>
+    </link>
+    <link name="base_link">
+        <inertial>
+            <mass value="0.0149878" />
+            <origin xyz="-3.78648e-18 -4.2386e-18 0.159" rpy="0 -0 0" />
+            <inertia ixx="0.000198722" ixy="0" ixz="0" iyy="0.000198722" iyz="0" izz="0.000374423" />
+        </inertial>
+        <visual>
+            <origin xyz="0 0 0" rpy="0 -0 0" />
+            <geometry>
+                <mesh filename="package://arips_description/meshes/base_link.stl" scale="1 1 1" />
             </geometry>
             <material name="0.756863_0.462745_0.109804_0.000000_0.000000">
@@ -23,49 +39,17 @@
         </visual>
     </link>
-    <link name="base_upper">
-        <inertial>
-            <mass value="0.00176738" />
-            <origin xyz="0.0388387 -0.0417081 0.36814" rpy="0 -0 0" />
-            <inertia ixx="0.000256556" ixy="6.74702e-06" ixz="-3.03595e-05" iyy="0.000255786" iyz="3.40732e-05" izz="4.45347e-05" />
-        </inertial>
-        <visual>
-            <origin xyz="0 0 0" rpy="0 -0 0" />
-            <geometry>
-                <mesh filename="package://arips_description/meshes/Base_upper.stl" scale="1 1 1" />
-            </geometry>
-            <material name="0.756863_0.462745_0.109804_0.000000_0.000000">
-                <color rgba="0.756863 0.462745 0.109804 1" />
-            </material>
-        </visual>
-    </link>
-    <link name="gripper">
-        <inertial>
-            <mass value="3.37196e-05" />
-            <origin xyz="-1.249e-16 -1.21431e-17 -0.0275681" rpy="0 -0 0" />
-            <inertia ixx="9.56595e-09" ixy="0" ixz="0" iyy="2.94892e-08" iyz="0" izz="2.11878e-08" />
-        </inertial>
-        <visual>
-            <origin xyz="0.07 -0.01 -0.456" rpy="0 -0 0" />
-            <geometry>
-                <mesh filename="package://arips_description/meshes/Gripper.stl" scale="1 1 1" />
-            </geometry>
-            <material name="0.647059_0.647059_0.647059_0.000000_0.000000">
-                <color rgba="0.647059 0.647059 0.647059 1" />
-            </material>
-        </visual>
-    </link>
-    <link name="kinect_beam">
-        <inertial>
-            <mass value="0.000375246" />
-            <origin xyz="-1.93985e-19 -0.651131 -6.66134e-16" rpy="0 -0 0" />
-            <inertia ixx="2.85294e-05" ixy="0" ixz="0" iyy="8.56168e-06" iyz="0" izz="1.99677e-05" />
-        </inertial>
-        <visual>
-            <origin xyz="0 0.1725 -1.442" rpy="0 -0 0" />
-            <geometry>
-                <mesh filename="package://arips_description/meshes/Kinect_beam.stl" scale="1 1 1" />
-            </geometry>
-            <material name="0.341176_0.776471_0.741176_0.000000_0.000000">
-                <color rgba="0.341176 0.776471 0.741176 0.1" />
+    <link name="door_gripper">
+        <inertial>
+            <mass value="0.000180456" />
+            <origin xyz="-1.64285e-18 -0.0248816 -4.02491e-17" rpy="0 -0 0" />
+            <inertia ixx="1.12954e-07" ixy="0" ixz="0" iyy="2.30182e-07" iyz="0" izz="1.83532e-07" />
+        </inertial>
+        <visual>
+            <origin xyz="0 -0.005 0" rpy="0 -0 0" />
+            <geometry>
+                <mesh filename="package://arips_description/meshes/Door_gripper.stl" scale="1 1 1" />
+            </geometry>
+            <material name="0.000000_0.588235_1.000000_0.000000_0.000000">
+                <color rgba="0 0.588235 1 1" />
             </material>
         </visual>
@@ -73,12 +57,12 @@
     <link name="kinect_mount">
         <inertial>
-            <mass value="0.000665142" />
-            <origin xyz="-0.01 -0.00127041 0.0491123" rpy="0 -0 0" />
-            <inertia ixx="3.39268e-07" ixy="0" ixz="0" iyy="3.54568e-06" iyz="7.50064e-10" izz="3.66293e-06" />
-        </inertial>
-        <visual>
-            <origin xyz="-0.01 0.14 -1.392" rpy="0 -0 0" />
-            <geometry>
-                <mesh filename="package://arips_description/meshes/kinect_mount.stl" scale="1 1 1" />
+            <mass value="0.00065" />
+            <origin xyz="0.0013 0.005 0.05" rpy="0 -0 0" />
+            <inertia ixx="3.52083e-06" ixy="0" ixz="0" iyy="3.14422e-07" iyz="0" izz="3.66192e-06" />
+        </inertial>
+        <visual>
+            <origin xyz="-0.14 0.005 -1.4114" rpy="0 -0 0" />
+            <geometry>
+                <mesh filename="package://arips_description/meshes/Kinect.stl" scale="1 1 1" />
             </geometry>
             <material name="0.156863_0.156863_0.156863_0.000000_0.000000">
@@ -87,17 +71,17 @@
         </visual>
     </link>
-    <link name="laptop">
-        <inertial>
-            <mass value="0.00232688" />
-            <origin xyz="0 2.94903e-17 -0.0125" rpy="0 -0 0" />
-            <inertia ixx="1.27299e-05" ixy="0" ixz="0" iyy="2.59544e-05" iyz="0" izz="3.84419e-05" />
-        </inertial>
-        <visual>
-            <origin xyz="0 -0.00848802 -0.201" rpy="0 -0 0" />
-            <geometry>
-                <mesh filename="package://arips_description/meshes/Laptop.stl" scale="1 1 1" />
-            </geometry>
-            <material name="0.156863_0.156863_0.156863_0.000000_0.000000">
-                <color rgba="0.156863 0.156863 0.156863 1" />
+    <link name="left_wheel">
+        <inertial>
+            <mass value="0.000190066" />
+            <origin xyz="0.1 0.155 0.055" rpy="0 -0 0" />
+            <inertia ixx="1.50073e-07" ixy="0" ixz="0" iyy="2.87475e-07" iyz="0" izz="1.50073e-07" />
+        </inertial>
+        <visual>
+            <origin xyz="0 0 0" rpy="0 -0 0" />
+            <geometry>
+                <mesh filename="package://arips_description/meshes/left_wheel.stl" scale="1 1 1" />
+            </geometry>
+            <material name="0.000000_0.588235_1.000000_0.000000_0.000000">
+                <color rgba="0 0.588235 1 1" />
             </material>
         </visual>
@@ -105,15 +89,15 @@
     <link name="link_0">
         <inertial>
-            <mass value="6e-05" />
-            <origin xyz="-0.0191667 -0.01 0.0125" rpy="0 -0 0" />
-            <inertia ixx="1.2125e-08" ixy="0" ixz="0" iyy="2.40833e-08" iyz="0" izz="2.99583e-08" />
-        </inertial>
-        <visual>
-            <origin xyz="-0.125 0.13 -0.676" rpy="0 -0 0" />
-            <geometry>
-                <mesh filename="package://arips_description/meshes/Link_0.stl" scale="1 1 1" />
-            </geometry>
-            <material name="0.498039_0.498039_0.498039_0.000000_0.000000">
-                <color rgba="0.498039 0.498039 0.498039 1" />
+            <mass value="0.000359788" />
+            <origin xyz="-0.02775 0.0035 0.037" rpy="0 -0 0" />
+            <inertia ixx="2.22229e-07" ixy="0" ixz="0" iyy="5.30275e-07" iyz="0" izz="4.24138e-07" />
+        </inertial>
+        <visual>
+            <origin xyz="0 0 -0.192" rpy="0 -0 0" />
+            <geometry>
+                <mesh filename="package://arips_description/meshes/link_0.stl" scale="1 1 1" />
+            </geometry>
+            <material name="0.000000_0.588235_1.000000_0.000000_0.000000">
+                <color rgba="0 0.588235 1 1" />
             </material>
         </visual>
@@ -121,15 +105,15 @@
     <link name="link_1">
         <inertial>
-            <mass value="5.80686e-05" />
-            <origin xyz="-0.085 8.32667e-17 -0.005" rpy="0 -0 0" />
-            <inertia ixx="4.70651e-09" ixy="0" ixz="0" iyy="1.82427e-07" iyz="0" izz="1.86166e-07" />
-        </inertial>
-        <visual>
-            <origin xyz="-0.1 0.14 -0.676" rpy="0 -0 0" />
-            <geometry>
-                <mesh filename="package://arips_description/meshes/Link_1.stl" scale="1 1 1" />
-            </geometry>
-            <material name="0.980392_0.713725_0.003922_0.000000_0.000000">
-                <color rgba="0.980392 0.713726 0.00392157 1" />
+            <mass value="0.0003603" />
+            <origin xyz="-0.0729 -6.73556e-19 -0.03355" rpy="0 -0 0" />
+            <inertia ixx="1.65931e-07" ixy="0" ixz="0" iyy="9.80594e-07" iyz="0" izz="8.76155e-07" />
+        </inertial>
+        <visual>
+            <origin xyz="0.0962 -6.73556e-19 -0.25755" rpy="0 -0 0" />
+            <geometry>
+                <mesh filename="package://arips_description/meshes/link_1.stl" scale="1 1 1" />
+            </geometry>
+            <material name="0.000000_0.588235_1.000000_0.000000_0.000000">
+                <color rgba="0 0.588235 1 1" />
             </material>
         </visual>
@@ -137,15 +121,15 @@
     <link name="link_2">
         <inertial>
-            <mass value="5.20686e-05" />
-            <origin xyz="-5.55112e-17 0.075 -0.005" rpy="0 -0 0" />
-            <inertia ixx="1.31717e-07" ixy="0" ixz="0" iyy="4.20651e-09" iyz="0" izz="1.35056e-07" />
-        </inertial>
-        <visual>
-            <origin xyz="0.07 0.14 -0.666" rpy="0 -0 0" />
-            <geometry>
-                <mesh filename="package://arips_description/meshes/Link_2.stl" scale="1 1 1" />
-            </geometry>
-            <material name="0.615686_0.811765_0.929412_0.000000_0.000000">
-                <color rgba="0.615686 0.811765 0.929412 1" />
+            <mass value="0.000317356" />
+            <origin xyz="-0.0629 -6.43626e-19 -0.03355" rpy="0 -0 0" />
+            <inertia ixx="1.46153e-07" ixy="0" ixz="0" iyy="6.96789e-07" iyz="0" izz="6.04797e-07" />
+        </inertial>
+        <visual>
+            <origin xyz="0.2662 -6.73556e-19 -0.25755" rpy="0 -0 0" />
+            <geometry>
+                <mesh filename="package://arips_description/meshes/link_2.stl" scale="1 1 1" />
+            </geometry>
+            <material name="0.000000_0.588235_1.000000_0.000000_0.000000">
+                <color rgba="0 0.588235 1 1" />
             </material>
         </visual>
@@ -153,126 +137,92 @@
     <link name="link_3">
         <inertial>
-            <mass value="0.000141372" />
-            <origin xyz="-9.71445e-17 -3.81639e-17 -0.1" rpy="0 -0 0" />
-            <inertia ixx="4.79191e-07" ixy="0" ixz="0" iyy="4.79191e-07" iyz="0" izz="1.59043e-08" />
-        </inertial>
-        <visual>
-            <origin xyz="0.07 -0.01 -0.656" rpy="0 -0 0" />
-            <geometry>
-                <mesh filename="package://arips_description/meshes/Link_3.stl" scale="1 1 1" />
-            </geometry>
-            <material name="0.647059_0.647059_0.647059_0.000000_0.000000">
-                <color rgba="0.647059 0.647059 0.647059 1" />
-            </material>
-        </visual>
-    </link>
-    <link name="base_footprint" />
-    <link name="wheel_left">
-        <inertial>
-            <mass value="7.85398e-05" />
-            <origin xyz="0.16 -0.092376 0.05" rpy="0 -0 0" />
-            <inertia ixx="9.81748e-08" ixy="0" ixz="0" iyy="4.97419e-08" iyz="0" izz="4.97419e-08" />
-        </inertial>
-        <visual>
-            <origin xyz="0 0 0" rpy="0 -0 0" />
-            <geometry>
-                <mesh filename="package://arips_description/meshes/Wheel_left.stl" scale="1 1 1" />
-            </geometry>
-            <material name="0.141176_0.694118_0.650980_0.000000_0.000000">
-                <color rgba="0.141176 0.694118 0.65098 1" />
-            </material>
-        </visual>
-    </link>
-    <link name="wheel_right">
-        <inertial>
-            <mass value="7.85398e-05" />
-            <origin xyz="-0.16 -0.092376 0.05" rpy="0 -0 0" />
-            <inertia ixx="9.81748e-08" ixy="0" ixz="0" iyy="4.97419e-08" iyz="0" izz="4.97419e-08" />
-        </inertial>
-        <visual>
-            <origin xyz="0 0 0" rpy="0 -0 0" />
-            <geometry>
-                <mesh filename="package://arips_description/meshes/Wheel_right.stl" scale="1 1 1" />
-            </geometry>
-            <material name="0.141176_0.694118_0.650980_0.000000_0.000000">
-                <color rgba="0.141176 0.694118 0.65098 1" />
-            </material>
-        </visual>
-    </link>
-    <joint name="fastened_1" type="fixed">
-        <origin xyz="-1.38778e-17 0 -0.2" rpy="-5.2711e-82 -3.08149e-33 3.42114e-49" />
+            <mass value="0.000135621" />
+            <origin xyz="5.55112e-17 -0.0227949 -0.031" rpy="0 -0 0" />
+            <inertia ixx="9.72341e-08" ixy="0" ixz="0" iyy="5.514e-08" iyz="0" izz="6.5486e-08" />
+        </inertial>
+        <visual>
+            <origin xyz="0.4162 4.57793e-17 -0.20595" rpy="0 -0 0" />
+            <geometry>
+                <mesh filename="package://arips_description/meshes/link_3.stl" scale="1 1 1" />
+            </geometry>
+            <material name="0.000000_0.588235_1.000000_0.000000_0.000000">
+                <color rgba="0 0.588235 1 1" />
+            </material>
+        </visual>
+    </link>
+    <link name="right_wheel">
+        <inertial>
+            <mass value="0.000190066" />
+            <origin xyz="0.1 -0.155 0.055" rpy="0 -0 0" />
+            <inertia ixx="1.50073e-07" ixy="0" ixz="0" iyy="2.87475e-07" iyz="0" izz="1.50073e-07" />
+        </inertial>
+        <visual>
+            <origin xyz="0 0 0" rpy="0 -0 0" />
+            <geometry>
+                <mesh filename="package://arips_description/meshes/right_wheel.stl" scale="1 1 1" />
+            </geometry>
+            <material name="0.000000_0.588235_1.000000_0.000000_0.000000">
+                <color rgba="0 0.588235 1 1" />
+            </material>
+        </visual>
+    </link>
+    <joint name="group_1_fastened_joint" type="fixed">
+        <origin xyz="0 0 0" rpy="0 -0 0" />
+        <axis xyz="-0 -0 -1" />
+        <parent link="base_link" />
+        <child link="left_wheel" />
+    </joint>
+    <joint name="group_1_fastened_joint_1" type="fixed">
+        <origin xyz="0 0 0" rpy="0 -0 0" />
+        <axis xyz="-0 -0 -1" />
+        <parent link="left_wheel" />
+        <child link="right_wheel" />
+    </joint>
+    <joint name="group_1_fastened_joint_2" type="fixed">
+        <origin xyz="0 0 0" rpy="0 -0 0" />
+        <axis xyz="-0 -0 -1" />
+        <parent link="right_wheel" />
+        <child link="alu" />
+    </joint>
+    <joint name="joint_2" type="revolute">
+        <origin xyz="-0.0962 2.77556e-17 0.06555" rpy="1.9945e-20 8.84458e-20 -5.55112e-17" />
         <axis xyz="0 0 1" />
-        <parent link="link_3" />
-        <child link="gripper" />
-    </joint>
-    <joint name="fastened_2" type="fixed">
-        <origin xyz="-0.01 -0.0325 0.05" rpy="5.55112e-17 -1.38667e-32 -3.04851e-32" />
-        <axis xyz="0 -1 0" />
-        <parent link="kinect_mount" />
-        <child link="kinect_beam" />
-    </joint>
-    <joint name="fastened_4" type="fixed">
-        <origin xyz="-0.000349049 0.000361977 0.176" rpy="3.14159 -0 0" />
-        <axis xyz="-0 -0 1" />
-        <parent link="base_upper" />
-        <child link="laptop" />
-    </joint>
-    <joint name="fastened_5" type="fixed">
-        <origin xyz="0 0 0" rpy="0 -0 0" />
-        <axis xyz="0 0 1" />
-        <parent link="base_lower" />
-        <child link="wheel_left" />
-    </joint>
-    <joint name="fastened_6" type="fixed">
-        <origin xyz="0 0 0" rpy="0 -0 0" />
-        <axis xyz="0 0 1" />
-        <parent link="base_lower" />
-        <child link="wheel_right" />
-    </joint>
-    <joint name="fastened_7" type="fixed">
-        <origin xyz="0 0 0" rpy="0 -0 0" />
-        <axis xyz="0 0 1" />
-        <parent link="base_lower" />
-        <child link="base_upper" />
-    </joint>
-    <joint name="fastened_8" type="fixed">
-        <origin xyz="0 0 0" rpy="0 -0 1.5708" />
-        <axis xyz="0 0 1" />
-        <parent link="base_footprint" />
-        <child link="base_lower" />
-    </joint>
-    <joint name="kinect_joint" type="continuous">
-        <origin xyz="0.01 -0.14 1.392" rpy="2.37643e-17 1.18821e-17 6.12323e-17" />
-        <axis xyz="-1 0 0" />
-        <parent link="base_upper" />
-        <child link="kinect_mount" />
-    </joint>
-    <joint name="revolute_2" type="revolute">
-        <origin xyz="-0.0191667 -0.01 0" rpy="0.0 0.0 0.0" />
-        <axis xyz="-0 -0 1" />
         <parent link="link_0" />
         <child link="link_1" />
-        <limit effort="1" velocity="1" lower="-2.3" upper="2.3" />
-    </joint>
-    <joint name="revolute_3" type="revolute">
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
Commit message: controller config for whole arm, all joints working

File: arips_description/urdf/arips.ros2_control.xacro (robot description, xacro)
@@ -147,6 +147,7 @@
                     <param name="max_position">0.871</param>
                     <param name="max_velocity_steps">3400</param>  <!-- Motor's max velocity in steps/s, model-dependent: STS3215=3400, STS3032=2900 (default: 3400) -->
-                    <param name="max_velocity">5.22</param>  <!-- Max velocity limit in rad/s (default: 5.22) -->
-                    <param name="position_center_steps">4095</param>  <!-- Motor step mapped to 0 rad: 0-4095 (default: 4095 → [0, 2π); set to 2048 for [−π, +π]) -->
+                    <param name="max_velocity">0.3</param>  <!-- Max velocity limit in rad/s (default: 5.22) -->
+                    <param name="position_center_steps">3730</param>  <!-- Motor step mapped to 0 rad: 0-4095 (default: 4095 → [0, 2π); set to 2048 for [−π, +π]) -->
+                    <param name="position_multiplicator">0.152226</param>  <!-- Multiplier for position conversion (default: 1.0) -->
                     <!-- Optional EEPROM parameters (omit any line to preserve the existing EEPROM value): -->
                     <!-- <param name="p_coefficient">32</param> -->   <!-- P gain (0-255): addr 21 (Mode 0) -->

File: arips_description/urdf/arips_onshape.urdf.xacro (robot description, xacro)
@@ -217,5 +217,5 @@
         <parent link="base_link" />
         <child link="link_0" />
-        <limit effort="1" velocity="1" lower="0.0" upper="6.2" />
+        <limit effort="1" velocity="1" lower="0.0" upper="0.871" />
     </joint>
     <joint name="kinect_joint" type="revolute">

Commit message: voice interface, arm simulation, lerobot record control node

File: arips_description/urdf/arips.ros2_control.xacro (robot description, xacro)
@@ -1,5 +1,5 @@
 <?xml version="1.0"?>
 <robot xmlns:xacro="http://www.ros.org/wiki/xacro">
-    <xacro:macro name="ros2_control_arips" params="serial_port baud_rate arm_enabled kinect_enabled">
+    <xacro:macro name="ros2_control_arips" params="serial_port baud_rate arm_enabled kinect_enabled enable_mock_mode">
         <ros2_control name="arips_servos" type="system">
             <hardware>
@@ -9,5 +9,5 @@
                 <param name="communication_timeout_ms">20</param>  <!-- Serial timeout: 1-1000 ms (default: 100) -->
                 <param name="use_sync_write">true</param>  <!-- Enable SyncWrite for multi-motor chains (default: true) -->
-                <param name="enable_mock_mode">false</param>  <!-- Simulation mode without hardware (default: false) -->
+                <param name="enable_mock_mode">${enable_mock_mode}</param>
                 <param name="reset_states_on_activate">"false"</param>  <!-- Reset position/velocity to zero on activation (default: true) -->
             </hardware>

File: arips_description/urdf/arips_onshape.urdf.xacro (robot description, xacro)
@@ -6,4 +6,5 @@
     <xacro:arg name="arm_enabled" default="true" />
     <xacro:arg name="kinect_enabled" default="true" />
+    <xacro:arg name="enable_mock_mode" default="false" />
     <xacro:include filename="$(find arips_description)/urdf/arips.ros2_control.xacro" />
     <link name="alu">
@@ -287,5 +288,5 @@
     </joint>
     <xacro:if value="$(arg use_ros2_control)">
-        <xacro:ros2_control_arips serial_port="$(arg serial_port)" baud_rate="$(arg baud_rate)" arm_enabled="$(arg arm_enabled)" kinect_enabled="$(arg kinect_enabled)" />
+        <xacro:ros2_control_arips serial_port="$(arg serial_port)" baud_rate="$(arg baud_rate)" arm_enabled="$(arg arm_enabled)" kinect_enabled="$(arg kinect_enabled)" enable_mock_mode="'$(arg enable_mock_mode)'" />
     </xacro:if>
 </robot>
