Commit message: switched description meshes from gltf to stl due to rendering bug, adaptations for ubuntu 26

File: arips_description/urdf/arips_onshape.urdf.xacro (robot description, xacro)
@@ -16,5 +16,5 @@
             <origin xyz="0 0 0" rpy="0 -0 0" />
             <geometry>
-                <mesh filename="package://arips_description/meshes/Base_lower.gltf" scale="1 1 1" />
+                <mesh filename="package://arips_description/meshes/Base_lower.stl" scale="1 1 1" />
             </geometry>
             <material name="0.756863_0.462745_0.109804_0.000000_0.000000">
@@ -32,5 +32,5 @@
             <origin xyz="0 0 0" rpy="0 -0 0" />
             <geometry>
-                <mesh filename="package://arips_description/meshes/Base_upper.gltf" scale="1 1 1" />
+                <mesh filename="package://arips_description/meshes/Base_upper.stl" scale="1 1 1" />
             </geometry>
             <material name="0.756863_0.462745_0.109804_0.000000_0.000000">
@@ -48,5 +48,5 @@
             <origin xyz="0.07 -0.01 -0.456" rpy="0 -0 0" />
             <geometry>
-                <mesh filename="package://arips_description/meshes/Gripper.gltf" scale="1 1 1" />
+                <mesh filename="package://arips_description/meshes/Gripper.stl" scale="1 1 1" />
             </geometry>
             <material name="0.647059_0.647059_0.647059_0.000000_0.000000">
@@ -64,5 +64,5 @@
             <origin xyz="0 0.1725 -1.442" rpy="0 -0 0" />
             <geometry>
-                <mesh filename="package://arips_description/meshes/Kinect_beam.gltf" scale="1 1 1" />
+                <mesh filename="package://arips_description/meshes/Kinect_beam.stl" scale="1 1 1" />
             </geometry>
             <material name="0.341176_0.776471_0.741176_0.000000_0.000000">
@@ -80,5 +80,5 @@
             <origin xyz="-0.01 0.14 -1.392" rpy="0 -0 0" />
             <geometry>
-                <mesh filename="package://arips_description/meshes/kinect_mount.gltf" scale="1 1 1" />
+                <mesh filename="package://arips_description/meshes/kinect_mount.stl" scale="1 1 1" />
             </geometry>
             <material name="0.156863_0.156863_0.156863_0.000000_0.000000">
@@ -96,5 +96,5 @@
             <origin xyz="0 -0.00848802 -0.201" rpy="0 -0 0" />
             <geometry>
-                <mesh filename="package://arips_description/meshes/Laptop.gltf" scale="1 1 1" />
+                <mesh filename="package://arips_description/meshes/Laptop.stl" scale="1 1 1" />
             </geometry>
             <material name="0.156863_0.156863_0.156863_0.000000_0.000000">
@@ -112,5 +112,5 @@
             <origin xyz="-0.125 0.13 -0.676" rpy="0 -0 0" />
             <geometry>
-                <mesh filename="package://arips_description/meshes/Link_0.gltf" scale="1 1 1" />
+                <mesh filename="package://arips_description/meshes/Link_0.stl" scale="1 1 1" />
             </geometry>
             <material name="0.498039_0.498039_0.498039_0.000000_0.000000">
@@ -128,5 +128,5 @@
             <origin xyz="-0.1 0.14 -0.676" rpy="0 -0 0" />
             <geometry>
-                <mesh filename="package://arips_description/meshes/Link_1.gltf" scale="1 1 1" />
+                <mesh filename="package://arips_description/meshes/Link_1.stl" scale="1 1 1" />
             </geometry>
             <material name="0.980392_0.713725_0.003922_0.000000_0.000000">
@@ -144,5 +144,5 @@
             <origin xyz="0.07 0.14 -0.666" rpy="0 -0 0" />
             <geometry>
-                <mesh filename="package://arips_description/meshes/Link_2.gltf" scale="1 1 1" />
+                <mesh filename="package://arips_description/meshes/Link_2.stl" scale="1 1 1" />
             </geometry>
             <material name="0.615686_0.811765_0.929412_0.000000_0.000000">
@@ -160,5 +160,5 @@
             <origin xyz="0.07 -0.01 -0.656" rpy="0 -0 0" />
             <geometry>
-                <mesh filename="package://arips_description/meshes/Link_3.gltf" scale="1 1 1" />
+                <mesh filename="package://arips_description/meshes/Link_3.stl" scale="1 1 1" />
             </geometry>
             <material name="0.647059_0.647059_0.647059_0.000000_0.000000">
@@ -177,5 +177,5 @@
             <origin xyz="0 0 0" rpy="0 -0 0" />
             <geometry>
-                <mesh filename="package://arips_description/meshes/Wheel_left.gltf" scale="1 1 1" />
+                <mesh filename="package://arips_description/meshes/Wheel_left.stl" scale="1 1 1" />
             </geometry>
             <material name="0.141176_0.694118_0.650980_0.000000_0.000000">
@@ -193,5 +193,5 @@
             <origin xyz="0 0 0" rpy="0 -0 0" />
             <geometry>
-                <mesh filename="package://arips_description/meshes/Wheel_right.gltf" scale="1 1 1" />
+                <mesh filename="package://arips_description/meshes/Wheel_right.stl" scale="1 1 1" />
             </geometry>
             <material name="0.141176_0.694118_0.650980_0.000000_0.000000">

Commit message: trajecory server accepts single point

File: arips_description/urdf/arips_onshape.urdf.xacro (robot description, xacro)
@@ -22,4 +22,10 @@
             </material>
         </visual>
+        <collision>
+            <origin xyz="0 0 0" rpy="0 -0 0" />
+            <geometry>
+                <mesh filename="package://arips_description/meshes/Alu.stl" scale="1 1 1" />
+            </geometry>
+        </collision>
     </link>
     <link name="base_link">
@@ -38,4 +44,10 @@
             </material>
         </visual>
+        <collision>
+            <origin xyz="0 0 0" rpy="0 -0 0" />
+            <geometry>
+                <mesh filename="package://arips_description/meshes/base_link.stl" scale="1 1 1" />
+            </geometry>
+        </collision>
     </link>
     <link name="door_gripper">
@@ -54,4 +66,10 @@
             </material>
         </visual>
+        <collision>
+            <origin xyz="0 -0.005 0" rpy="0 -0 0" />
+            <geometry>
+                <mesh filename="package://arips_description/meshes/Door_gripper.stl" scale="1 1 1" />
+            </geometry>
+        </collision>
     </link>
     <link name="kinect_mount">
@@ -70,4 +88,10 @@
             </material>
         </visual>
+        <collision>
+            <origin xyz="-0.14 0.005 -1.4114" rpy="0 -0 0" />
+            <geometry>
+                <mesh filename="package://arips_description/meshes/Kinect.stl" scale="1 1 1" />
+            </geometry>
+        </collision>
     </link>
     <link name="left_wheel">
@@ -86,4 +110,10 @@
             </material>
         </visual>
+        <collision>
+            <origin xyz="0 0 0" rpy="0 -0 0" />
+            <geometry>
+                <mesh filename="package://arips_description/meshes/left_wheel.stl" scale="1 1 1" />
+            </geometry>
+        </collision>
     </link>
     <link name="link_0">
@@ -102,4 +132,10 @@
             </material>
         </visual>
+        <collision>
+            <origin xyz="0 0 -0.192" rpy="0 -0 0" />
+            <geometry>
+                <mesh filename="package://arips_description/meshes/link_0.stl" scale="1 1 1" />
+            </geometry>
+        </collision>
     </link>
     <link name="link_1">
@@ -118,4 +154,10 @@
             </material>
         </visual>
+        <collision>
+            <origin xyz="0.0962 -6.73556e-19 -0.25755" rpy="0 -0 0" />
+            <geometry>
+                <mesh filename="package://arips_description/meshes/link_1.stl" scale="1 1 1" />
+            </geometry>
+        </collision>
     </link>
     <link name="link_2">
@@ -134,4 +176,10 @@
             </material>
         </visual>
+        <collision>
+            <origin xyz="0.2662 -6.73556e-19 -0.25755" rpy="0 -0 0" />
+            <geometry>
+                <mesh filename="package://arips_description/meshes/link_2.stl" scale="1 1 1" />
+            </geometry>
+        </collision>
     </link>
     <link name="link_3">
@@ -150,4 +198,10 @@
             </material>
         </visual>
+        <collision>
+            <origin xyz="0.4162 4.57793e-17 -0.20595" rpy="0 -0 0" />
+            <geometry>
+                <mesh filename="package://arips_description/meshes/link_3.stl" scale="1 1 1" />
+            </geometry>
+        </collision>
     </link>
     <link name="right_wheel">
@@ -166,4 +220,10 @@
             </material>
         </visual>
+        <collision>
+            <origin xyz="0 0 0" rpy="0 -0 0" />
+            <geometry>
+                <mesh filename="package://arips_description/meshes/right_wheel.stl" scale="1 1 1" />
+            </geometry>
+        </collision>
     </link>
     <joint name="group_1_fastened_joint" type="fixed">

Commit message: better and smoother arm teleop

File: arips_description/urdf/arips_onshape.urdf.xacro (robot description, xacro)
@@ -251,5 +251,5 @@
         <parent link="link_0" />
         <child link="link_1" />
-        <limit effort="1" velocity="1" lower="-2.26893" upper="2.26893" />
+        <limit effort="1" velocity="2" lower="-2.26893" upper="2.26893" />
     </joint>
     <joint name="joint_3" type="revolute">
@@ -258,5 +258,5 @@
         <parent link="link_1" />
         <child link="link_2" />
-        <limit effort="1" velocity="1" lower="-2.44346" upper="2.44346" />
+        <limit effort="1" velocity="2" lower="-2.44346" upper="2.44346" />
     </joint>
     <joint name="joint_4" type="revolute">
@@ -265,5 +265,5 @@
         <parent link="link_2" />
         <child link="link_3" />
-        <limit effort="1" velocity="1" lower="-2.0944" upper="2.0944" />
+        <limit effort="1" velocity="2" lower="-2.44346" upper="2.44346" />
     </joint>
     <joint name="joint_door_gripper" type="continuous">
@@ -278,5 +278,5 @@
         <parent link="base_link" />
         <child link="link_0" />
-        <limit effort="1" velocity="1" lower="0.0" upper="0.871" />
+        <limit effort="1" velocity="0.2" lower="0.0" upper="0.871" />
     </joint>
     <joint name="kinect_joint" type="revolute">
