Commit message: teleop node for leader arm

File: arips_leader_arm/urdf/leader_arm.urdf.xacro (robot description, xacro)
@@ -51,5 +51,5 @@
     </joint>
   </xacro:macro>
-  <link name="base_plate">
+  <link name="leader_base_plate">
     <visual>
       <origin xyz="0 0 ${base_thickness / 2}"/>
@@ -62,6 +62,6 @@
     </collision>
   </link>
-  <!-- link_1: cylinder rotating about the vertical axis -->
-  <link name="link_1">
+  <!-- leader_link_1: cylinder rotating about the vertical axis -->
+  <link name="leader_link_1">
     <visual>
       <origin xyz="0 0 ${link_1_length / 2}"/>
@@ -74,18 +74,18 @@
     </collision>
   </link>
-  <xacro:revolute_joint name="leader_joint_1" parent="base_plate" child="link_1"
+  <xacro:revolute_joint name="leader_joint_1" parent="leader_base_plate" child="leader_link_1"
                         xyz="0 0 ${base_thickness}" axis="0 0 1"/>
-  <xacro:box_link name="link_2" length="${link_2_length}" material="orange"/>
-  <xacro:revolute_joint name="leader_joint_2" parent="link_1" child="link_2"
+  <xacro:box_link name="leader_link_2" length="${link_2_length}" material="orange"/>
+  <xacro:revolute_joint name="leader_joint_2" parent="leader_link_1" child="leader_link_2"
                         xyz="0 0 ${link_1_length}" axis="0 1 0"/>
-  <xacro:box_link name="link_3" length="${link_3_length}" material="blue"/>
-  <xacro:revolute_joint name="leader_joint_3" parent="link_2" child="link_3"
+  <xacro:box_link name="leader_link_3" length="${link_3_length}" material="blue"/>
+  <xacro:revolute_joint name="leader_joint_3" parent="leader_link_2" child="leader_link_3"
                         xyz="0 ${link_y_offset} ${link_2_length}" axis="0 1 0"/>
-  <!-- URDF mimic supports a single source joint, so keeping link_4 upright
+  <!-- URDF mimic supports a single source joint, so keeping leader_link_4 upright
        (q2 + q3 + q4 = 0) takes two chained mimic joints: joint_4 = -q2, joint_4b = -q3 -->
-  <link name="link_4_helper"/>
+  <link name="leader_link_4_helper"/>
   <joint name="leader_joint_virtual" type="revolute">
-    <parent link="link_3"/>
-    <child link="link_4_helper"/>
+    <parent link="leader_link_3"/>
+    <child link="leader_link_4_helper"/>
     <origin xyz="0 ${-link_y_offset} ${link_3_length}"/>
     <axis xyz="0 1 0"/>
@@ -93,18 +93,18 @@
     <mimic joint="leader_joint_2" multiplier="-1" offset="0"/>
   </joint>
-  <xacro:box_link name="link_4" length="${link_4_length}" material="orange"/>
+  <xacro:box_link name="leader_link_4" length="${link_4_length}" material="orange"/>
   <joint name="leader_joint_virtual_b" type="revolute">
-    <parent link="link_4_helper"/>
-    <child link="link_4"/>
+    <parent link="leader_link_4_helper"/>
+    <child link="leader_link_4"/>
     <axis xyz="0 1 0"/>
     <limit lower="${-2 * pi}" upper="${2 * pi}" effort="${joint_effort}" velocity="${joint_velocity}"/>
     <mimic joint="leader_joint_3" multiplier="-1" offset="3.14159"/>
   </joint>
-  <!-- link_4 points down, so its local +z (end of link) is downward.
+  <!-- leader_link_4 points down, so its local +z (end of link) is downward.
        joint_4 rotates about the link axis, joint_gripper about the horizontal x axis. -->
-  <xacro:box_link name="link_5" length="${link_5_length}" material="blue"/>
-  <xacro:revolute_joint name="leader_joint_4" parent="link_4" child="link_5"
+  <xacro:box_link name="leader_link_5" length="${link_5_length}" material="blue"/>
+  <xacro:revolute_joint name="leader_joint_4" parent="leader_link_4" child="leader_link_5"
                         xyz="0 0 ${link_4_length}" axis="0 0 1"/>
-  <link name="link_gripper">
+  <link name="leader_link_gripper">
     <visual>
       <origin xyz="-${gripper_thickness} 0 0"/>
@@ -117,5 +117,5 @@
     </collision>
   </link>
-  <xacro:revolute_joint name="leader_joint_gripper" parent="link_5" child="link_gripper"
+  <xacro:revolute_joint name="leader_joint_gripper" parent="leader_link_5" child="leader_link_gripper"
                         xyz="0 0 ${link_5_length}" axis="-1 0 0"/>
 </robot>
